Commit message: feat(h_i controller):add the basic protocol of LK_MF9025

File: src/warrior_description/ros2_control/warrior.ros2_control.xacro (robot description, xacro)
@@ -47,5 +47,4 @@
       <hardware>
         <plugin>warrior_hardware/ImuHardwareInterface</plugin>
-        <param name="imu_id">1025</param>
       </hardware>
       <sensor name="imu">
@@ -54,4 +53,38 @@
         <state_interface name="roll"/>
       </sensor>
+      <joint name="left_9025">
+        <command_interface name="position">
+          <param name="min">-1</param>
+          <param name="max">1</param>
+        </command_interface>
+        <command_interface name="velocity">
+          <param name="min">-1</param>
+          <param name="max">1</param>
+        </command_interface>
+        <command_interface name="moment">
+          <param name="min">-1</param>
+          <param name="max">1</param>
+        </command_interface>
+        <state_interface name="position"/>
+        <state_interface name="velocity"/>
+        <state_interface name="acceleration"/>
+      </joint>
+      <joint name="right_9025">
+        <command_interface name="position">
+          <param name="min">-1</param>
+          <param name="max">1</param>
+        </command_interface>
+        <command_interface name="velocity">
+          <param name="min">-1</param>
+          <param name="max">1</param>
+        </command_interface>
+        <command_interface name="moment">
+          <param name="min">-1</param>
+          <param name="max">1</param>
+        </command_interface>
+        <state_interface name="position"/>
+        <state_interface name="velocity"/>
+        <state_interface name="acceleration"/>
+      </joint>
     </ros2_control>
   </xacro:macro>

Commit message: feat(h_i controller):finish the go1 hardware_interface and controller rudiment

File: src/warrior_description/ros2_control/warrior.ros2_control.xacro (robot description, xacro)
@@ -44,5 +44,5 @@
       </joint>
     </ros2_control>
-    <ros2_control name="imu_hardware" type="system">
+    <ros2_control name="can_hardware" type="system">
       <hardware>
         <plugin>warrior_hardware/ImuHardwareInterface</plugin>
@@ -88,4 +88,77 @@
       </joint>
     </ros2_control>
+    <ros2_control name="serialport" type="system">
+      <hardware>
+        <plugin>warrior_hardware/SerialPorttHardwareInterface</plugin>
+      </hardware>
+      <joint name="Go1_LF">
+        <command_interface name="position">
+          <param name="min">-1</param>
+          <param name="max">1</param>
+        </command_interface>
+        <command_interface name="velocity">
+          <param name="min">-1</param>
+          <param name="max">1</param>
+        </command_interface>
+        <command_interface name="moment">
+          <param name="min">-1</param>
+          <param name="max">1</param>
+        </command_interface>
+        <state_interface name="position"/>
+        <state_interface name="velocity"/>
+        <state_interface name="acceleration"/>
+      </joint>
+      <joint name="Go1_LB">
+        <command_interface name="position">
+          <param name="min">-1</param>
+          <param name="max">1</param>
+        </command_interface>
+        <command_interface name="velocity">
+          <param name="min">-1</param>
+          <param name="max">1</param>
+        </command_interface>
+        <command_interface name="moment">
+          <param name="min">-1</param>
+          <param name="max">1</param>
+        </command_interface>
+        <state_interface name="position"/>
+        <state_interface name="velocity"/>
+        <state_interface name="acceleration"/>
+      </joint>
+      <joint name="Go1_RF">
+        <command_interface name="position">
+          <param name="min">-1</param>
+          <param name="max">1</param>
+        </command_interface>
+        <command_interface name="velocity">
+          <param name="min">-1</param>
+          <param name="max">1</param>
+        </command_interface>
+        <command_interface name="moment">
+          <param name="min">-1</param>
+          <param name="max">1</param>
+        </command_interface>
+        <state_interface name="position"/>
+        <state_interface name="velocity"/>
+        <state_interface name="acceleration"/>
+      </joint>
+      <joint name="Go1_RB">
+        <command_interface name="position">
+          <param name="min">-1</param>
+          <param name="max">1</param>
+        </command_interface>
+        <command_interface name="velocity">
+          <param name="min">-1</param>
+          <param name="max">1</param>
+        </command_interface>
+        <command_interface name="moment">
+          <param name="min">-1</param>
+          <param name="max">1</param>
+        </command_interface>
+        <state_interface name="position"/>
+        <state_interface name="velocity"/>
+        <state_interface name="acceleration"/>
+      </joint>
+    </ros2_control>
   </xacro:macro>
 </robot>

Commit message: style(h_i):separate imu from can_hardware_interface.

File: src/warrior_description/ros2_control/warrior.ros2_control.xacro (robot description, xacro)
@@ -47,4 +47,169 @@
       <hardware>
         <plugin>warrior_hardware/MF9025HardwareInterface</plugin>
+      </hardware>
+      <!-- <sensor name="imu">
+        <state_interface name="pitch"/>
+        <state_interface name="yaw"/>
+        <state_interface name="roll"/>
+      </sensor> -->
+      <joint name="left_9025">
+        <command_interface name="position">
+          <param name="min">-1</param>
+          <param name="max">1</param>
+        </command_interface>
+        <command_interface name="velocity">
+          <param name="min">-1</param>
+          <param name="max">1</param>
+        </command_interface>
+        <command_interface name="torque">
+          <param name="min">-1</param>
+          <param name="max">1</param>
+        </command_interface>
+        <state_interface name="position"/>
+        <state_interface name="velocity"/>
+        <state_interface name="torque"/>
+      </joint>
+      <joint name="right_9025">
+        <command_interface name="position">
+          <param name="min">-1</param>
+          <param name="max">1</param>
+        </command_interface>
+        <command_interface name="velocity">
+          <param name="min">-1</param>
+          <param name="max">1</param>
+        </command_interface>
+        <command_interface name="torque">
+          <param name="min">-1</param>
+          <param name="max">1</param>
+        </command_interface>
+        <state_interface name="position"/>
+        <state_interface name="velocity"/>
+        <state_interface name="torque"/>
+      </joint>
+    </ros2_control>
+    <ros2_control name="serialport" type="system">
+      <hardware>
+        <plugin>warrior_hardware/Go1HardwareInterface</plugin>
+      </hardware>
+      <joint name="Go1_LF">
+        <command_interface name="position">
+          <param name="min">-1</param>
+          <param name="max">1</param>
+        </command_interface>
+        <command_interface name="velocity">
+          <param name="min">-1</param>
+          <param name="max">1</param>
+        </command_interface>
+        <command_interface name="torque">
+          <param name="min">-1</param>
+          <param name="max">1</param>
+        </command_interface>
+        <command_interface name="damp">
+        <param name="min">-1</param>
+        <param name="max">1</param>
+        </command_interface>
+        <command_interface name="zero_torque">
+          <param name="min">-1</param>
+          <param name="max">1</param>
+        </command_interface>
+        <command_interface name="torque_and_position">
+          <param name="min">-1</param>
+          <param name="max">1</param>
+        </command_interface>
+        <state_interface name="position"/>
+        <state_interface name="velocity"/>
+        <state_interface name="acceleration"/>
+      </joint>
+      <joint name="Go1_LB">
+        <command_interface name="position">
+          <param name="min">-1</param>
+          <param name="max">1</param>
+        </command_interface>
+        <command_interface name="velocity">
+          <param name="min">-1</param>
+          <param name="max">1</param>
+        </command_interface>
+        <command_interface name="torque">
+          <param name="min">-1</param>
+          <param name="max">1</param>
+        </command_interface>
+        <command_interface name="damp">
+        <param name="min">-1</param>
+        <param name="max">1</param>
+        </command_interface>
+        <command_interface name="zero_torque">
+          <param name="min">-1</param>
+          <param name="max">1</param>
+        </command_interface>
+        <command_interface name="torque_and_position">
+          <param name="min">-1</param>
+          <param name="max">1</param>
+        </command_interface>
+        <state_interface name="position"/>
+        <state_interface name="velocity"/>
+        <state_interface name="acceleration"/>
+      </joint>
+      <joint name="Go1_RF">
+        <command_interface name="position">
+          <param name="min">-1</param>
+          <param name="max">1</param>
+        </command_interface>
+        <command_interface name="velocity">
+          <param name="min">-1</param>
+          <param name="max">1</param>
+        </command_interface>
+        <command_interface name="torque">
+          <param name="min">-1</param>
+          <param name="max">1</param>
+        </command_interface>
+        <command_interface name="damp">
+        <param name="min">-1</param>
+        <param name="max">1</param>
+        </command_interface>
+        <command_interface name="zero_torque">
+          <param name="min">-1</param>
+          <param name="max">1</param>
+        </command_interface>
+        <command_interface name="torque_and_position">
+          <param name="min">-1</param>
+          <param name="max">1</param>
+        </command_interface>
+        <state_interface name="position"/>
+        <state_interface name="velocity"/>
+        <state_interface name="acceleration"/>
+      </joint>
+      <joint name="Go1_RB">
+        <command_interface name="position">
+          <param name="min">-1</param>
+          <param name="max">1</param>
+        </command_interface>
+        <command_interface name="velocity">
+          <param name="min">-1</param>
+          <param name="max">1</param>
+        </command_interface>
+        <command_interface name="torque">
+          <param name="min">-1</param>
+          <param name="max">1</param>
+        </command_interface>
+        <command_interface name="damp">
+        <param name="min">-1</param>
+        <param name="max">1</param>
+        </command_interface>
+        <command_interface name="zero_torque">
+          <param name="min">-1</param>
+          <param name="max">1</param>
+        </command_interface>
+        <command_interface name="torque_and_position">
+          <param name="min">-1</param>
+          <param name="max">1</param>
+        </command_interface>
+        <state_interface name="position"/>
+        <state_interface name="velocity"/>
+        <state_interface name="acceleration"/>
+      </joint>
+    </ros2_control>
+      <ros2_control name="imu_hardware" type="sensor">
+      <hardware>
+        <plugin>warrior_hardware/ImuHardwareInterface</plugin>
       </hardware>
       <sensor name="imu">
@@ -53,159 +218,4 @@
         <state_interface name="roll"/>
       </sensor>
-      <joint name="left_9025">
-        <command_interface name="position">
-          <param name="min">-1</param>
-          <param name="max">1</param>
-        </command_interface>
-        <command_interface name="velocity">
-          <param name="min">-1</param>
-          <param name="max">1</param>
-        </command_interface>
-        <command_interface name="torque">
-          <param name="min">-1</param>
-          <param name="max">1</param>
-        </command_interface>
-        <state_interface name="position"/>
-        <state_interface name="velocity"/>
-        <state_interface name="torque"/>
-      </joint>
-      <joint name="right_9025">
-        <command_interface name="position">
-          <param name="min">-1</param>
-          <param name="max">1</param>
-        </command_interface>
-        <command_interface name="velocity">
-          <param name="min">-1</param>
-          <param name="max">1</param>
-        </command_interface>
-        <command_interface name="torque">
-          <param name="min">-1</param>
-          <param name="max">1</param>
-        </command_interface>
-        <state_interface name="position"/>
-        <state_interface name="velocity"/>
-        <state_interface name="torque"/>
-      </joint>
-    </ros2_control>
-    <ros2_control name="serialport" type="system">
-      <hardware>
-        <plugin>warrior_hardware/Go1HardwareInterface</plugin>
-      </hardware>
-      <joint name="Go1_LF">
-        <command_interface name="position">
-          <param name="min">-1</param>
-          <param name="max">1</param>
-        </command_interface>
-        <command_interface name="velocity">
-          <param name="min">-1</param>
-          <param name="max">1</param>
-        </command_interface>
-        <command_interface name="torque">
-          <param name="min">-1</param>
-          <param name="max">1</param>
-        </command_interface>
-        <command_interface name="damp">
-        <param name="min">-1</param>
-        <param name="max">1</param>
-        </command_interface>
-        <command_interface name="zero_torque">
-          <param name="min">-1</param>
-          <param name="max">1</param>
-        </command_interface>
-        <command_interface name="torque_and_position">
-          <param name="min">-1</param>
-          <param name="max">1</param>
-        </command_interface>
-        <state_interface name="position"/>
-        <state_interface name="velocity"/>
-        <state_interface name="acceleration"/>
-      </joint>
-      <joint name="Go1_LB">
-        <command_interface name="position">
-          <param name="min">-1</param>
-          <param name="max">1</param>
-        </command_interface>
-        <command_interface name="velocity">
-          <param name="min">-1</param>
-          <param name="max">1</param>
-        </command_interface>
-        <command_interface name="torque">
-          <param name="min">-1</param>
-          <param name="max">1</param>
-        </command_interface>
-        <command_interface name="damp">
-        <param name="min">-1</param>
-        <param name="max">1</param>
-        </command_interface>
-        <command_interface name="zero_torque">
-          <param name="min">-1</param>
-          <param name="max">1</param>
-        </command_interface>
-        <command_interface name="torque_and_position">
-          <param name="min">-1</param>
-          <param name="max">1</param>
-        </command_interface>
-        <state_interface name="position"/>
-        <state_interface name="velocity"/>
-        <state_interface name="acceleration"/>
-      </joint>
-      <joint name="Go1_RF">
-        <command_interface name="position">
-          <param name="min">-1</param>
-          <param name="max">1</param>
-        </command_interface>
-        <command_interface name="velocity">
-          <param name="min">-1</param>
-          <param name="max">1</param>
-        </command_interface>
-        <command_interface name="torque">
-          <param name="min">-1</param>
-          <param name="max">1</param>
-        </command_interface>
-        <command_interface name="damp">
-        <param name="min">-1</param>
-        <param name="max">1</param>
-        </command_interface>
-        <command_interface name="zero_torque">
-          <param name="min">-1</param>
-          <param name="max">1</param>
-        </command_interface>
-        <command_interface name="torque_and_position">
-          <param name="min">-1</param>
-          <param name="max">1</param>
-        </command_interface>
-        <state_interface name="position"/>
-        <state_interface name="velocity"/>
-        <state_interface name="acceleration"/>
-      </joint>
-      <joint name="Go1_RB">
-        <command_interface name="position">
-          <param name="min">-1</param>
-          <param name="max">1</param>
-        </command_interface>
-        <command_interface name="velocity">
-          <param name="min">-1</param>
-          <param name="max">1</param>
-        </command_interface>
-        <command_interface name="torque">
-          <param name="min">-1</param>
-          <param name="max">1</param>
-        </command_interface>
-        <command_interface name="damp">
-        <param name="min">-1</param>
-        <param name="max">1</param>
-        </command_interface>
-        <command_interface name="zero_torque">
-          <param name="min">-1</param>
-          <param name="max">1</param>
-        </command_interface>
-        <command_interface name="torque_and_position">
-          <param name="min">-1</param>
-          <param name="max">1</param>
-        </command_interface>
-        <state_interface name="position"/>
-        <state_interface name="velocity"/>
-        <state_interface name="acceleration"/>
-      </joint>
     </ros2_control>
   </xacro:macro>
